File: MacroDecKnob [PCB]/MacroDecKnob.kicad_pcb (KiCad board)
At the start: 2 copper layers, 176.9 x 106.9 mm, 37 parts, among them J1 Batt, J2 Mounting Hole, J3 Mounting Hole, J4 Mounting Hole, J5 Mounting Hole, J6 Mounting Hole, J7 5V-ARGB, SW1 SW_Push, SW10 SW_Push, SW11 SW_Push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

Commit message: upgrade 2"display
display 320x 240 upgrade
Connections:
- R6 pad 1: Net-(J1-Pin_2) -> Net-(J1-Pin_1)
Routing:
- net Net-(J1-Pin_1): track 26.3 -> 33.7 mm
- net Net-(J1-Pin_2): track 25.7 -> 19.7 mm
Changed lines of the file:
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@@
 		)
 		(property "Value" "5V-ARGB"
-			(at 0 7.41 0)
+			(at 3.1926 2.7288 90)
 			(layer "F.Fab")
 			(effects
@@
 			(at 0 0.5 0)
 			(unlocked yes)
-			(layer "F.SilkS")
+			(layer "F.Fab")
 			(effects
 				(font
@@
 		(attr through_hole)
 		(fp_rect
-			(start 1.17 4.6)
-			(end 10.07 9)
+			(start -12.1 -9.3)
+			(end 12.2 9.4)
 			(stroke
 				(width 0.1)
@@
 		)
 		(fp_rect
-			(start -11.8 -9)
-			(end 11.8 9)
+			(start -12 -9.2)
+			(end 12 9.2)
+			(stroke
+				(width 0.05)
+				(type solid)
+			)
+			(fill no)
+			(layer "F.CrtYd")
+		)
+		(fp_rect
+			(start 1.17 4.6)
+			(end 10.07 9)
 			(stroke
 				(width 0.1)
@@
 			)
 			(fill no)
-			(layer "F.SilkS")
+			(layer "F.Fab")
 		)
 		(fp_rect
-			(start -12 -9.2)
-			(end 12 9.2)
+			(start -11.8 -9)
+			(end 11.8 9)
 			(stroke
-				(width 0.05)
+				(width 0.1)
 				(type solid)
 			)
 			(fill no)
-			(layer "F.CrtYd")
+			(layer "F.Fab")
 		)
-		(fp_text user "USB-C"
-			(at 8.128 6.7564 0)
+		(fp_text user "${REFERENCE}"
+			(at 0 -2.5 0)
 			(unlocked yes)
-			(layer "F.SilkS")
+			(layer "F.Fab")
 			(effects
 				(font
 					(size 1 1)
-					(thickness 0.1)
+					(thickness 0.15)
 				)
-				(justify left bottom)
 			)
 		)
-		(fp_text user "${REFERENCE}"
-			(at 0 -2.5 0)
+		(fp_text user "USB-C"
+			(at 8.128 6.7564 0)
 			(unlocked yes)
 			(layer "F.Fab")
@@
 				(font
 					(size 1 1)
-					(thickness 0.15)
+					(thickness 0.1)
 				)
+				(justify left bottom)
 			)
 		)
@@
 			(roundrect_rratio 0.15)
 			(net 29 "Net-(J1-Pin_1)")
-			(pinfunction "B-")
+			(pinfunction "B+")
 			(pintype "power_out")
 			(thermal_bridge_angle 45)
@@
 			(roundrect_rratio 0.15)
 			(net 28 "Net-(J1-Pin_2)")
-			(pinfunction "B+")
+			(pinfunction "B-")
 			(pintype "power_out")
 			(thermal_bridge_angle 45)
@@
 		)
 		(property "Value" "ON-OFF"
-			(at -2.8254 8.5058 90)
+			(at -6.6556 4.198 180)
 			(layer "F.Fab")
 			(effects
@@
 			(layers "*.Cu" "*.Mask")
 			(remove_unused_layers no)
-			(net 28 "Net-(J1-Pin_2)")
+			(net 29 "Net-(J1-Pin_1)")
 			(pintype "passive")
 		)
@@
 	)
 	(segment
-		(start 59.756513 70.890702)
-		(end 60.129413 70.517802)
-		(width 0.8)
-		(layer "B.Cu")
-		(net 28)
-	)
-	(segment
 		(start 60.0964 66.212189)
 		(end 60.129413 66.245202)
@@
 	)
 	(segment
-		(start 60.129413 70.517802)
-		(end 60.129413 66.245202)
-		(width 0.8)
-		(layer "B.Cu")
-		(net 28)
-	)
-	(segment
 		(start 65.8854 51.996)
 		(end 60.0964 57.785)
@@
 	)
 	(segment
-		(start 58.608113 70.890702)
-		(end 59.756513 70.890702)
-		(width 0.8)
-		(layer "B.Cu")
-		(net 28)
-	)
-	(segment
 		(start 77.4512 51.996)
 		(end 77.4512 53.4604)
@@
 	)
 	(segment
+		(start 60.434298 70.890702)
+		(end 62.629413 68.695587)
+		(width 0.8)
+		(layer "B.Cu")
+		(net 29)
+	)
+	(segment
 		(start 77.4512 53.4604)
 		(end 76.454 54.4576)
@@
 	)
 	(segment
+		(start 62.629413 68.695587)
+		(end 62.629413 66.245202)
+		(width 0.8)
+		(layer "B.Cu")
+		(net 29)
+	)
+	(segment
 		(start 76.454 54.4576)
 		(end 66.3702 54.4576)
@@
 		(width 0.8)
 		(layer "B.Cu")
+		(net 29)
+	)
+	(segment
+		(start 58.608113 70.890702)
+		(end 60.434298 70.890702)
+		(width 0.8)
+		(layer "B.Cu")
